Commit message: refactoring file directory and add grip and release

File: resource/m0609_gripper2.urdf (robot description, URDF)
Before this commit: robot m0609, 11 links, 10 joints
Links:
- removed link rg2_hand
- removed link rg2_leftfinger
- removed link rg2_rightfinger
- added link hand_link, mass 1.684558; collision mesh filename=package://rg2_meshes/collision/RG2_Hand_col.STL; visual mesh filename=package://rg2_meshes/visual/RG2_Hand_vis.STL
- added link l_finger_link, mass 0.081638; collision mesh filename=package://rg2_meshes/collision/RG2_LeftFinger_col.STL; visual mesh filename=package://rg2_meshes/visual/RG2_LeftFinger_vis.STL
- added link l_moment_arm_link, mass 0.160209; collision mesh filename=package://rg2_meshes/collision/RG2_LeftMomentArm_col.STL; visual mesh filename=package://rg2_meshes/visual/RG2_LeftMomentArm_vis.STL
- added link r_finger_link, mass 0.081637; collision mesh filename=package://rg2_meshes/collision/RG2_RightFinger_col.STL; visual mesh filename=package://rg2_meshes/visual/RG2_RightFinger_vis.STL
- added link r_moment_arm_link, mass 0.160209; collision mesh filename=package://rg2_meshes/collision/RG2_RightMomentArm_col.STL; visual mesh filename=package://rg2_meshes/visual/RG2_RightMomentArm_vis.STL
Joints:
- removed joint rg2_finger_joint1
- removed joint rg2_finger_joint2
- removed joint ur5_hand_joint
- added joint base_fixed_joint: type fixed, parent link_6, child hand_link, origin xyz=0.000 0.000 0.000 rpy=0 -1.571 0
- added joint l_finger_1_joint: type revolute, parent hand_link, child l_moment_arm_link, origin xyz=0.105 0.017 0.010 rpy=0 0 0, axis 0 0 1, limit lower=-0.45 upper=0.45 effort=10.6 velocity=3.14
- added joint l_finger_2_joint: type revolute, parent l_moment_arm_link, child l_finger_link, origin xyz=0.049 0.026 0.000 rpy=0 0 0, axis 0 0 1, limit lower=-0.45 upper=0.45 effort=10.6 velocity=3.14
- added joint r_finger_1_joint: type revolute, parent hand_link, child r_moment_arm_link, origin xyz=0.105 -0.017 0.010 rpy=0 0 0, axis 0 0 1, limit lower=-0.45 upper=0.45 effort=10.6 velocity=3.14
- added joint r_finger_2_joint: type revolute, parent r_moment_arm_link, child r_finger_link, origin xyz=0.049 -0.026 0.000 rpy=0 0 0, axis 0 0 1, limit lower=-0.45 upper=0.45 effort=10.6 velocity=3.14
