Commit message: minimized robot.urdf

File: quadruped_controller_cpp/src/champ/champ_base/resource/robot.urdf (robot description, URDF)
Before this commit: robot go2, 19 links, 18 joints
Links:
- link base_link: geometry 
- link imu_link: geometry collision box size=.001 .001 .001
- link lf_foot_link: geometry collision sphere radius=0.02
- link lf_hip_link: geometry collision cylinder length=0.04 radius=0.046
- link lf_lower_leg_link: geometry collision box size=0.213 0.016 0.016
- link lf_upper_leg_link: geometry collision box size=0.213 0.0245 0.034
- link lh_foot_link: geometry collision sphere radius=0.02
- link lh_hip_link: geometry collision cylinder length=0.04 radius=0.046
- link lh_lower_leg_link: geometry collision box size=0.213 0.016 0.016
- link lh_upper_leg_link: geometry collision box size=0.213 0.0245 0.034
- link rf_foot_link: geometry collision sphere radius=0.02
- link rf_hip_link: geometry collision cylinder length=0.04 radius=0.046
- link rf_lower_leg_link: geometry collision box size=0.213 0.016 0.016
- link rf_upper_leg_link: geometry collision box size=0.213 0.0245 0.034
- link rh_foot_link: geometry collision sphere radius=0.02
- link rh_hip_link: geometry collision cylinder length=0.04 radius=0.046
- link rh_lower_leg_link: geometry collision box size=0.213 0.016 0.016
- link rh_upper_leg_link: geometry collision box size=0.213 0.0245 0.034
- link trunk: geometry collision box size=0.3762 0.0935 0.114
